File: device/hardware/fsk-timekeeper.kicad_sch (KiCad schematic)
At the start: 22 parts, among them J1 SENSOR, SW1 SW_SPST, U1 SuperMini nRF52840, U2 Ai-Thinker Ra-01SH, U3 TPS61040DBV, U4 ATGM336H

Commit message: fix: leave the Ra-01SH TXEN and RXEN pins unconnected
The Ra-01SH ties TXEN to the SX1262 DIO2 through a 0 ohm resistor and
leaves RXEN open, and RadioLib's begin() already makes DIO2 drive the RF
switch. Driving TXEN from P1.04 fought DIO2 at the start and end of every
transmission, and RXEN reached nothing. The schematic and board drop both
nets, and the firmware drops setRfSwitchPins() and the pin definitions.

The board also carries the refilled GND zone, the bottom +BATT trace
moved to y = 125 mm, and the J1 and SW1 values synced from the schematic.

Co-Authored-By: Claude Opus 5.5 <noreply@anthropic.com>
Connections:
- net RXEN: no longer names the net of U1.8 (P0.24)
- net RXEN: no longer U2.11 (DIO5)
- net TXEN: no longer names the net of U1.11 (P1.04-LF)
- net TXEN: no longer U2.5 (DIO0)
- no-connect marks 13 -> 17
Changed lines of the file:
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@@
+	)
+	(no_connect
+		(at 48.26 99.06)
 	)
 	(no_connect
@@
 	)
 	(no_connect
+		(at 132.08 81.28)
+	)
+	(no_connect
 		(at 86.36 83.82)
 	)
@@
 	)
 	(no_connect
+		(at 48.26 91.44)
+	)
+	(no_connect
 		(at 132.08 76.2)
 	)
@@
 	(no_connect
 		(at 132.08 86.36)
+	)
+	(no_connect
+		(at 132.08 93.98)
 	)
 	(no_connect
@@
 		)
 	)
-	(label "TXEN"
-		(at 48.26 99.06 180)
-		(effects
-			(font
-				(size 1.27 1.27)
-			)
-			(justify right bottom)
-		)
-	)
 	(label "SENSE"
 		(at 80.01 127 0)
@@
 		)
 	)
-	(label "RXEN"
-		(at 48.26 91.44 180)
-		(effects
-			(font
-				(size 1.27 1.27)
-			)
-			(justify right bottom)
-		)
-	)
 	(label "SCK"
 		(at 48.26 88.9 180)
@@
 		)
 	)
-	(label "TXEN"
-		(at 132.08 81.28 0)
-		(effects
-			(font
-				(size 1.27 1.27)
-			)
-			(justify left bottom)
-		)
-	)
 	(label "SENSOR"
 		(at 57.15 127 180)
@@
 		)
 	)
-	(label "RXEN"
-		(at 132.08 93.98 0)
-		(effects
-			(font
-				(size 1.27 1.27)
-			)
-			(justify left bottom)
-		)
-	)

Commit message: fix: keep hand-soldered parts out of the JLCPCB BOM and CPL
BT1, J1, L1, SW1, U2 and U4 have no LCSC number but still went into the
BOM and CPL, and U1 into the CPL, so JLCPCB would list them as unmatched
lines. Their symbols and footprints are now excluded from the BOM and
position files, and the assembly plugin's project.db follows.

Co-Authored-By: Claude Opus 5.5 <noreply@anthropic.com>
Parts:
- BT1, J1, L1, SW1, U2, U4: now left out of the parts list
Changed lines of the file:
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@@
 		(body_style 1)
 		(exclude_from_sim no)
-		(in_bom yes)
+		(in_bom no)
 		(on_board yes)
-		(in_pos_files yes)
+		(in_pos_files no)
 		(dnp no)
 		(fields_autoplaced yes)
@@
 		(in_bom no)
 		(on_board yes)
-		(in_pos_files yes)
+		(in_pos_files no)
 		(dnp no)
 		(fields_autoplaced yes)
@@
 		(body_style 1)
 		(exclude_from_sim no)
-		(in_bom yes)
+		(in_bom no)
 		(on_board yes)
-		(in_pos_files yes)
+		(in_pos_files no)
 		(dnp no)
 		(fields_autoplaced yes)
@@
 		(body_style 1)
 		(exclude_from_sim no)
-		(in_bom yes)
+		(in_bom no)
 		(on_board yes)
-		(in_pos_files yes)
+		(in_pos_files no)
 		(dnp no)
 		(fields_autoplaced yes)
@@
 		(body_style 1)
 		(exclude_from_sim no)
-		(in_bom yes)
+		(in_bom no)
 		(on_board yes)
-		(in_pos_files yes)
+		(in_pos_files no)
 		(dnp no)
 		(property "Reference" "U4"
@@
 		(body_style 1)
 		(exclude_from_sim no)
-		(in_bom yes)
+		(in_bom no)
 		(on_board yes)
-		(in_pos_files yes)
+		(in_pos_files no)
 		(dnp no)
 		(fields_autoplaced yes)
@@
 		(body_style 1)
 		(exclude_from_sim no)
-		(in_bom yes)
+		(in_bom no)
 		(on_board yes)
-		(in_pos_files yes)
+		(in_pos_files no)
 		(dnp no)
 		(property "Reference" "SW1"
