File: device/hardware/fsk-timekeeper.kicad_sch (KiCad schematic)
At the start: 22 parts, among them J1 SENSOR, SW1 SW_SPST, U1 SuperMini nRF52840, U2 Ai-Thinker Ra-01SH, U3 TPS61040DBV, U4 ATGM336H

Commit message: fix(hardware): refine power routing and refresh fabrication files
Parts:
- SW1: value SW_SPST -> POWER
Changed lines of the file:
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@@
 			)
 		)
-		(property "Value" "SW_SPST"
+		(property "Value" "POWER"
 			(at 238.76 120.6499 90)
 			(hide yes)
