File: device/hardware/fsk-timekeeper.kicad_sch (KiCad schematic)
At the start: 22 parts, among them J1 SENSOR, SW1 POWER, U1 SuperMini nRF52840, U2 Ai-Thinker Ra-01SH, U3 TPS61040DBV, U4 ATGM336H

Commit message: feat(hardware): route the camera trigger to J1 pin 2
J1 pin 2 was not connected. It now carries TRIG from U1 pin 17 (P0.31),
the line trigger the camera master drives (PIN_CAMERA_TRIG). Sensor
harnesses leave it unconnected.

- Schematic: TRIG labels at J1 pin 2 and U1 pin 17 replace the no-connect
  flags.
- PCB: TRIG routed, one more GND via; no footprint moved. The silkscreen
  marks pin 2 TRIG instead of x and resizes the J1, PPS and URL labels.
- Gerbers, drill files and the JLCPCB production files regenerated.

Co-Authored-By: Claude Opus 5.5 <noreply@anthropic.com>
Connections:
- net TRIG: now reaches J1.2 (Pin_2)
- net TRIG: now also U1.17 (P0.31-LF)
- no-connect marks 17 -> 15
Changed lines of the file:
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@@
-	)
-	(no_connect
-		(at 86.36 83.82)
 	)
 	(no_connect
@@
 	(no_connect
 		(at 132.08 93.98)
-	)
-	(no_connect
-		(at 199.39 124.46)
 	)
 	(no_connect
@@
 		)
 	)
+	(label "TRIG"
+		(at 86.36 83.82 0)
+		(effects
+			(font
+				(size 1.27 1.27)
+			)
+			(justify left bottom)
+		)
+	)
 	(label "MOSI"
 		(at 48.26 83.82 180)
@@
 		(effects
 			(font
+				(size 1.27 1.27)
+			)
+			(justify right bottom)
+		)
+	)
+	(label "TRIG"
+		(at 199.39 124.46 180)
+		(effects
+			(font
